File: hw/thermal.sch (KiCad schematic (older format))
At the start: 30 parts, among them IC1 ATTINY2313-P, J1 USB_2, J2 RJ12, J3 DB9, J4 JACK_2P, Q1 TIP120, Q2 TIP120, U1 LM7805, U2 LTV847, X1 12MHz

Commit message: Cleanup hw dir
Parts:
- removed Q1, Q2: TIP120, symbol NPN
- added Q1, Q2: IRL530N, ~, symbol MOSFET_N
- added R15, R16: 100k, symbol R
Connections:
- net labels added: FAN1, FAN2
- wire segments 129 -> 128
Other:
- moved on the sheet: R13, R14
